Commit message: retained original names for robot and joints

File: mycobot_320pi/urdf/mycobot_320pi_2022.urdf (robot description, URDF)
Before this commit: robot mycobot_320pi_with_gripper, 8 links, 7 joints
Joints:
- removed joint joint_1
- removed joint joint_2
- removed joint joint_3
- removed joint joint_4
- removed joint joint_5
- removed joint joint_6
- added joint joint2_to_joint1: type revolute, parent base, child link1, origin xyz=0 0 0.162 rpy=0 0 0, axis 0 0 1, limit lower=-2.96 upper=2.96 effort=1000.0 velocity=0
- added joint joint3_to_joint2: type revolute, parent link1, child link2, origin xyz=0 0 0 rpy=0 -1.5708 1.5708, axis 0 0 1, limit lower=-2.79 upper=2.79 effort=1000.0 velocity=0
- added joint joint4_to_joint3: type revolute, parent link2, child link3, origin xyz=0.13635 0 0    rpy=0 0 0, axis  0 0 1, limit lower=-2.79 upper=2.79 effort=1000.0 velocity=0
- added joint joint5_to_joint4: type revolute, parent link3, child link4, origin xyz=0.1205 0 0.082  rpy= 0 0 1.57080, axis  0 0 1, limit lower=-2.79 upper=2.79 effort=1000.0 velocity=0
- added joint joint6_to_joint5: type revolute, parent link4, child link5, origin xyz=0 -0.084 0 rpy=1.5708 0 0, axis 0 0 1, limit lower=-2.96 upper=2.96 effort=1000.0 velocity=0
- added joint joint6output_to_joint6: type revolute, parent link5, child link6, origin xyz=0 0.06635 0 rpy=-1.5708 0 0, axis 0 0 1, limit lower=-3.05 upper=3.05 effort=1000.0 velocity=0

File: mycobot_320pi/urdf/mycobot_320pi_2022_gripper.urdf (robot description, URDF)
Before this commit: robot mycobot_320pi_with_gripper, 15 links, 14 joints
Links:
- added link tcp
Joints:
- removed joint joint_1
- removed joint joint_2
- removed joint joint_3
- removed joint joint_4
- removed joint joint_5
- removed joint joint_6
- added joint joint2_to_joint1: type revolute, parent base, child link1, origin xyz=0 0 0.162 rpy=0 0 0, axis 0 0 1, limit lower=-2.96 upper=2.96 effort=1000.0 velocity=0
- added joint joint3_to_joint2: type revolute, parent link1, child link2, origin xyz=0 0 0 rpy=0 -1.5708 1.5708, axis 0 0 1, limit lower=-2.79 upper=2.79 effort=1000.0 velocity=0
- added joint joint4_to_joint3: type revolute, parent link2, child link3, origin xyz=0.13635 0 0    rpy=0 0 0, axis  0 0 1, limit lower=-2.79 upper=2.79 effort=1000.0 velocity=0
- added joint joint5_to_joint4: type revolute, parent link3, child link4, origin xyz=0.1205 0 0.082  rpy= 0 0 1.57080, axis  0 0 1, limit lower=-2.79 upper=2.79 effort=1000.0 velocity=0
- added joint joint6_to_joint5: type revolute, parent link4, child link5, origin xyz=0 -0.084 0 rpy=1.5708 0 0, axis 0 0 1, limit lower=-2.96 upper=2.96 effort=1000.0 velocity=0
- added joint joint6output_to_joint6: type revolute, parent link5, child link6, origin xyz=0 0.06635 0 rpy=-1.5708 0 0, axis 0 0 1, limit lower=-3.05 upper=3.05 effort=1000.0 velocity=0
- added joint tcp_jnt: type fixed, parent gripper_base, child tcp, origin xyz=0 0.1125 -0.018 rpy=0 0 0

File: mycobot_320pi_moveit_config/config/firefighter.ros2_control.xacro (robot description, xacro)
@@ -1,5 +1,5 @@
 <?xml version="1.0"?>
 <robot xmlns:xacro="http://www.ros.org/wiki/xacro">
-    <xacro:macro name="mycobot_320pi_with_gripper_ros2_control" params="name initial_positions_file">
+    <xacro:macro name="firefighter_ros2_control" params="name initial_positions_file">
         <xacro:property name="initial_positions" value="${load_yaml(initial_positions_file)['initial_positions']}"/>
         <ros2_control name="${name}" type="system">
@@ -8,43 +8,43 @@
                 <plugin>mock_components/GenericSystem</plugin>
             </hardware>
-            <joint name="joint_1">
+            <joint name="joint2_to_joint1">
                 <command_interface name="position"/>
                 <state_interface name="position">
-                  <param name="initial_value">${initial_positions['joint_1']}</param>
+                  <param name="initial_value">${initial_positions['joint2_to_joint1']}</param>
                 </state_interface>
                 <state_interface name="velocity"/>
             </joint>
-            <joint name="joint_2">
+            <joint name="joint3_to_joint2">
                 <command_interface name="position"/>
                 <state_interface name="position">
-                  <param name="initial_value">${initial_positions['joint_2']}</param>
+                  <param name="initial_value">${initial_positions['joint3_to_joint2']}</param>
                 </state_interface>
                 <state_interface name="velocity"/>
             </joint>
-            <joint name="joint_3">
+            <joint name="joint4_to_joint3">
                 <command_interface name="position"/>
                 <state_interface name="position">
-                  <param name="initial_value">${initial_positions['joint_3']}</param>
+                  <param name="initial_value">${initial_positions['joint4_to_joint3']}</param>
                 </state_interface>
                 <state_interface name="velocity"/>
             </joint>
-            <joint name="joint_4">
+            <joint name="joint5_to_joint4">
                 <command_interface name="position"/>
                 <state_interface name="position">
-                  <param name="initial_value">${initial_positions['joint_4']}</param>
+                  <param name="initial_value">${initial_positions['joint5_to_joint4']}</param>
                 </state_interface>
                 <state_interface name="velocity"/>
             </joint>
-            <joint name="joint_5">
+            <joint name="joint6_to_joint5">
                 <command_interface name="position"/>
                 <state_interface name="position">
-                  <param name="initial_value">${initial_positions['joint_5']}</param>
+                  <param name="initial_value">${initial_positions['joint6_to_joint5']}</param>
                 </state_interface>
                 <state_interface name="velocity"/>
             </joint>
-            <joint name="joint_6">
+            <joint name="joint6output_to_joint6">
                 <command_interface name="position"/>
                 <state_interface name="position">
-                  <param name="initial_value">${initial_positions['joint_6']}</param>
+                  <param name="initial_value">${initial_positions['joint6output_to_joint6']}</param>
                 </state_interface>
                 <state_interface name="velocity"/>
