Commit message: updated gripper urdf and moveit config files

File: mycobot_320pi/urdf/mycobot_320pi_2022_gripper.urdf (robot description, URDF)
Before this commit: robot firefighter, 16 links, 15 joints
Joints:
- removed joint mycobot_gripper_joint
- added joint gripper_controller: type revolute, parent gripper_base, child gripper_left3, origin xyz=-0.018 0.016 0 rpy=0 0 0, axis 0 0 1, limit lower=-0.7 upper=0.3 effort=1000.0 velocity=0
- joint gripper_base_to_gripper_left2_mimic_jnt: limit lower=-0.8 upper=0.5 effort=1000.0 velocity=0 -> lower=-0.8 upper=0.8 effort=1000.0 velocity=0; mimic joint=mycobot_gripper_joint multiplier=1.0 offset=0 -> joint=gripper_controller multiplier=1.0 offset=0
- joint gripper_base_to_gripper_right2_mimic_jnt: limit lower=-0.5 upper=0.8 effort=1000.0 velocity=0 -> lower=-0.8 upper=0.8 effort=1000.0 velocity=0; mimic joint=mycobot_gripper_joint multiplier=-1.0 offset=0 -> joint=gripper_controller multiplier=-1.0 offset=0
- joint gripper_base_to_gripper_right3_mimic_jnt: limit lower=-0.3 upper=0.7 effort=1000.0 velocity=0 -> lower=-0.8 upper=0.8 effort=1000.0 velocity=0; mimic joint=mycobot_gripper_joint multiplier=-1.0 offset=0 -> joint=gripper_controller multiplier=-1.0 offset=0
- joint gripper_left3_to_gripper_left1_mimic_jnt: limit lower=-0.5 upper=0.5 effort=1000.0 velocity=0 -> lower=-0.8 upper=0.8 effort=1000.0 velocity=0; mimic joint=mycobot_gripper_joint multiplier=-1.0 offset=0 -> joint=gripper_controller multiplier=-1.0 offset=0
- joint gripper_right3_to_gripper_right1_mimic_jnt: limit lower=-0.5 upper=0.5 effort=1000.0 velocity=0 -> lower=-0.8 upper=0.8 effort=1000.0 velocity=0; mimic joint=mycobot_gripper_joint multiplier=1.0 offset=0 -> joint=gripper_controller multiplier=1.0 offset=0
- joint tcp_jnt: origin xyz=0 0.1125 -0.018 rpy=0 0 0 -> xyz=0 0.0145 0.1465 rpy=0 0 -1.5708; parent gripper_base -> link6

File: mycobot_320pi_moveit_config/config/firefighter.ros2_control.xacro (robot description, xacro)
@@ -50,8 +50,8 @@
                 <state_interface name="velocity"/>
             </joint>
-            <joint name="mycobot_gripper_joint">
+            <joint name="gripper_controller">
                 <command_interface name="position"/>
                 <state_interface name="position">
-                  <param name="initial_value">${initial_positions['mycobot_gripper_joint']}</param>
+                  <param name="initial_value">${initial_positions['gripper_controller']}</param>
                 </state_interface>
                 <state_interface name="velocity"/>
